File: ESP32_KitTesla/ESP32_DevKit/ESP32_DevKit.kicad_pcb (KiCad board)
At the start: 2 copper layers, 29 x 58 mm, 28 parts, among them J1 SM04B-SRSS-TB(LF)(SN), J2 Conn_01x19_Pin, J3 Conn_01x19_Pin, P1 USB_C_Plug, Q1 MMBT2222ALT1G, Q2 MMBT2222ALT1G, U1 AP2112K-3.3TRG1, U2 CH340C, U3 ESP32-WROVER-E

Commit message: ESP32_terminado
Parts:
- removed D3: WS2812B, LED_SMD:LED_WS2812B_PLCC4_5.0x5.0mm_P3.2mm
- added D4: IR26-21C_L110_TR8, LED_SMD:LED_1206_3216Metric_Pad1.42x1.75mm_HandSolder, F.Cu at (192.3, 79.6)
- added R7: 80, Resistor_SMD:R_0805_2012Metric_Pad1.20x1.40mm_HandSolder, F.Cu at (192.5, 77.0)
- moved REF** 1.10 mm to (203.0, 48.4)
Connections:
- BT pad 5: (no net) -> unconnected-(S1-Pad5)
- RST pad 5: (no net) -> unconnected-(S2-Pad5)
Routing:
- net VBUS: track 52.6 -> 79.5 mm, vias 2 -> 5
- net /GPIO25: track 37.4 -> 13.7 mm
- net GNDREF: track 70.3 -> 76.6 mm, vias 15 -> 16
- net /GPIO0: track 79.7 -> 75.1 mm
- net Net-(D4-K): track 0.00 -> 2.67 mm
